File: testSchematic.sch (EAGLE design)
At the start: 43 parts, among them T1 TIP122, U1 ESP12ESMD

Commit message: esp connectivity
Parts:
- removed OK1, OK2, OK3, OK4, OK5, OK6, OK7, OK8: PC817, optocoupler:PC817
- removed R10, R11, R12, R13, R14, R15, R16, R5, R6, R7, R8, R9: (no value), rcl:R-EU_0204/7
- removed X1, X2, X3, X4, X5, X6, X7, X8: (no value), con-wago-500:W237-102
- added C1: 100uF, capacitor-wima:C2,5-3
- added FLASH, RESET: (no value), switch-omron:10-XX
- added OK10, OK11, OK12, OK13, OK14, OK15, OK16, OK9: PC817, optocoupler:PC817
- added R18, R20, R22, R24, R26, R28, R30, R32: 1k, rcl:R-EU_0204/7
- added R19, R21, R23, R25, R27, R29, R31, R33: (no value), rcl:R-EU_0204/7
- added X10, X11, X12, X13, X14, X15, X16, X17: (no value), con-wago-500:W237-102
- R1, R2, R3, R4: value (none) -> 10k; device rcl:R-EU_0204/7 -> rcl:R-EU_0207/10
- R17: value (none) -> 1k
Connections:
- removed net N$10: OK5.A, R9.1
- removed net N$11: R9.2, X5-2.KL
- removed net N$12: OK6.A, R11.1
- removed net N$13: R11.2, X6-2.KL
- removed net N$14: OK7.A, R13.1
- removed net N$15: R13.2, X7-2.KL
- removed net N$16: OK8.A, R15.1
- removed net N$17: R15.2, X8-2.KL
- removed net N$20: R1.2, X1-2.KL
- removed net N$7: R5.2, X3-2.KL
- removed net N$8: OK4.A, R7.1
- removed net N$9: R7.2, X4-2.KL
- new net N$21: OK9.A, R18.1
- new net N$22: R18.2, X10-2.KL
- new net N$23: OK10.A, R20.1
- new net N$24: R20.2, X11-2.KL
- new net N$25: OK11.A, R22.1
- new net N$26: R22.2, X12-2.KL
- new net N$27: OK12.A, R24.1
- new net N$28: R24.2, X13-2.KL
- new net N$29: OK13.A, R26.1
- new net N$30: R26.2, X14-2.KL
- new net N$31: OK14.A, R28.1
- new net N$32: R28.2, X15-2.KL
- new net N$33: OK15.A, R30.1
- new net N$34: R30.2, X16-2.KL
- new net N$35: OK16.A, R32.1
- new net N$36: R32.2, X17-2.KL
- new net PA2_BP_TX2: U1.RX
- new net PA3_BP_RX2: U1.TX
- net +12V: now also X10-1.KL, X11-1.KL, X12-1.KL, X13-1.KL, X14-1.KL, X15-1.KL, X16-1.KL, X17-1.KL; no longer X1-1.KL, X2-1.KL, X3-1.KL, X4-1.KL, X5-1.KL, X6-1.KL, X7-1.KL, X8-1.KL
- net +3V3: now also C1.2, R1.2, R19.1, R2.2, R21.1, R23.1, R25.1, R27.1, R29.1, R3.2, R31.1, R33.1, U1.VCC; no longer R10.1, R12.1, R14.1, R16.1, R2.1, R4.1, R6.1, R8.1
- net GND: now also C1.1, FLASH.S1, OK10.C, OK10.EMIT, OK11.C, OK11.EMIT, OK12.C, OK12.EMIT, OK13.C, OK13.EMIT, OK14.C, OK14.EMIT, OK15.C, OK15.EMIT, OK16.C, OK16.EMIT, OK9.C, OK9.EMIT, R4.1, RESET.P, U1.GND; no longer OK1.C, OK1.EMIT, OK2.C, OK2.EMIT, OK3.C, OK3.EMIT, OK4.C, OK4.EMIT, OK5.C, OK5.EMIT, OK6.C, OK6.EMIT, OK7.C, OK7.EMIT, OK8.C, OK8.EMIT
- net N$3: now also R1.1, RESET.S, U1.RESET; no longer OK2.A, R3.1
- net N$4: now also R2.1, U1.CH_PD; no longer R3.2, X2-2.KL
- net N$5: now also R4.2, U1.GPIO15; no longer OK1.A, R1.1
- net N$6: now also FLASH.P1, R3.1, U1.GPIO0; no longer OK3.A, R5.1
- net UCTLR_PIN_: now also OK10.COL, OK11.COL, OK12.COL, OK13.COL, OK14.COL, OK15.COL, OK16.COL, OK9.COL, R19.2, R21.2, R23.2, R25.2, R27.2, R29.2, R31.2, R33.2; no longer OK1.COL, OK2.COL, OK3.COL, OK4.COL, OK5.COL, OK6.COL, OK7.COL, OK8.COL, R10.2, R12.2, R14.2, R16.2, R2.2, R4.2, R6.2, R8.2
